File: modules/CpuRamModule/CpuRamModule.kicad_pcb (KiCad board)
At the start: 4 copper layers, 67.3 x 59.1 mm, 16 parts, among them J1 Conn_02x20_Odd_Even, SW1 SW_Push, SW2 SW_DIP_x04, U2 Z80CPU, U3 SST39SF010

Commit message: Update
Routing:
- net VCC: track 238.9 -> 231.2 mm
- net BRQ: track 129.6 -> 130.1 mm
Changed lines of the file:
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@@
     (effects (font (size 1 1) (thickness 0.15)))
   )
-  (segment (start 68.625 77.92) (end 69.85 76.695) (width 0.25) (layer "F.Cu") (net 1))
-  (segment (start 66.925 78.579009) (end 67.584009 77.92) (width 0.25) (layer "F.Cu") (net 1))
-  (segment (start 67.584009 77.92) (end 68.625 77.92) (width 0.25) (layer "F.Cu") (net 1))
-  (segment (start 69.85 76.695) (end 69.85 63.065) (width 0.25) (layer "F.Cu") (net 1))
+  (segment (start 106.68 53.95) (end 106.68 46.355) (width 0.25) (layer "F.Cu") (net 1))
   (segment (start 114.9775 76.8575) (end 114.9775 70.495) (width 0.25) (layer "F.Cu") (net 1))
-  (segment (start 66.925 79.510991) (end 66.925 78.579009) (width 0.25) (layer "F.Cu") (net 1))
   (segment (start 117.475 79.355) (end 114.9775 76.8575) (width 0.25) (layer "F.Cu") (net 1))
-  (segment (start 69.85 63.065) (end 68.05 61.265) (width 0.25) (layer "F.Cu") (net 1))
-  (segment (start 66.979505 79.565495) (end 66.925 79.510991) (width 0.25) (layer "F.Cu") (net 1))
-  (segment (start 62.23 84.315) (end 66.979505 79.565495) (width 0.25) (layer "F.Cu") (net 1))
+  (segment (start 106.68 54.5775) (end 106.68 53.95) (width 0.25) (layer "In1.Cu") (net 1))
+  (segment (start 114.9775 62.875) (end 106.68 54.5775) (width 0.25) (layer "In1.Cu") (net 1))
   (segment (start 62.23 84.315) (end 63.165 85.25) (width 0.25) (layer "In2.Cu") (net 1))
   (segment (start 68.05 61.265) (end 69.175 60.14) (width 0.25) (layer "In2.Cu") (net 1))
@@
   (segment (start 87.45 82.095) (end 87.45 73.965) (width 0.25) (layer "B.Cu") (net 2))
   (segment (start 84.055 85.49) (end 87.45 82.095) (width 0.25) (layer "B.Cu") (net 2))
+  (segment (start 60.865 80.41) (end 58.82 80.41) (width 0.25) (layer "F.Cu") (net 3))
+  (segment (start 57.785 79.375) (end 57.785 53.79) (width 0.25) (layer "F.Cu") (net 3))
+  (segment (start 58.915 52.66) (end 63.955 52.66) (width 0.25) (layer "F.Cu") (net 3))
   (segment (start 62.23 81.775) (end 60.865 80.41) (width 0.25) (layer "F.Cu") (net 3))
-  (segment (start 58.915 52.66) (end 63.955 52.66) (width 0.25) (layer "F.Cu") (net 3))
-  (segment (start 58.235 53.34) (end 58.915 52.66) (width 0.25) (layer "F.Cu") (net 3))
-  (segment (start 58.235 79.825) (end 58.235 53.34) (width 0.25) (layer "F.Cu") (net 3))
-  (segment (start 60.865 80.41) (end 58.82 80.41) (width 0.25) (layer "F.Cu") (net 3))
-  (segment (start 68.05 48.565) (end 63.955 52.66) (width 0.25) (layer "F.Cu") (net 3))
-  (segment (start 58.82 80.41) (end 58.235 79.825) (width 0.25) (layer "F.Cu") (net 3))
+  (segment (start 58.82 80.41) (end 57.785 79.375) (width 0.25) (layer "F.Cu") (net 3))
+  (segment (start 63.955 52.66) (end 68.05 48.565) (width 0.25) (layer "F.Cu") (net 3))
+  (segment (start 57.785 53.79) (end 58.915 52.66) (width 0.25) (layer "F.Cu") (net 3))
   (segment (start 118.6 79.885) (end 118.6 50.655) (width 0.25) (layer "F.Cu") (net 4))
   (segment (start 114.375 84.11) (end 118.6 79.885) (width 0.25) (layer "F.Cu") (net 4))
@@
   (segment (start 85.91 87.445) (end 98.265 75.09) (width 0.25) (layer "In1.Cu") (net 38))
   (segment (start 84.455 75.13) (end 83.29 73.965) (width 0.25) (layer "F.Cu") (net 39))
+  (segment (start 60.865 50.12) (end 59.203299 50.12) (width 0.25) (layer "F.Cu") (net 39))
+  (segment (start 59.203299 50.12) (end 57.15 52.173299) (width 0.25) (layer "F.Cu") (net 39))
   (segment (start 104.575 75.13) (end 113.8525 65.8525) (width 0.25) (layer "F.Cu") (net 39))
   (segment (start 113.8525 55.847069) (end 115.57 54.129569) (width 0.25) (layer "F.Cu") (net 39))
+  (segment (start 82.645991 86.36) (end 84.455 84.550991) (width 0.25) (layer "F.Cu") (net 39))
+  (segment (start 57.15 84.455) (end 59.055 86.36) (width 0.25) (layer "F.Cu") (net 39))
+  (segment (start 113.8525 65.8525) (end 113.8525 55.847069) (width 0.25) (layer "F.Cu") (net 39))
   (segment (start 59.055 86.36) (end 82.645991 86.36) (width 0.25) (layer "F.Cu") (net 39))
-  (segment (start 57.785 85.09) (end 59.055 86.36) (width 0.25) (layer "F.Cu") (net 39))
-  (segment (start 113.8525 65.8525) (end 113.8525 55.847069) (width 0.25) (layer "F.Cu") (net 39))
+  (segment (start 84.455 75.13) (end 104.575 75.13) (width 0.25) (layer "F.Cu") (net 39))
+  (segment (start 62.23 48.755) (end 60.865 50.12) (width 0.25) (layer "F.Cu") (net 39))
+  (segment (start 115.57 54.129569) (end 115.57 50.165) (width 0.25) (layer "F.Cu") (net 39))
+  (segment (start 57.15 52.173299) (end 57.15 84.455) (width 0.25) (layer "F.Cu") (net 39))
+  (segment (start 115.57 50.165) (end 114.3 48.895) (width 0.25) (layer "F.Cu") (net 39))
   (segment (start 84.455 84.550991) (end 84.455 75.13) (width 0.25) (layer "F.Cu") (net 39))
-  (segment (start 84.455 75.13) (end 104.575 75.13) (width 0.25) (layer "F.Cu") (net 39))
-  (segment (start 57.785 51.538299) (end 57.785 85.09) (width 0.25) (layer "F.Cu") (net 39))
-  (segment (start 115.57 54.129569) (end 115.57 50.165) (width 0.25) (layer "F.Cu") (net 39))
-  (segment (start 62.23 48.755) (end 60.865 50.12) (width 0.25) (layer "F.Cu") (net 39))
-  (segment (start 115.57 50.165) (end 114.3 48.895) (width 0.25) (layer "F.Cu") (net 39))
-  (segment (start 82.645991 86.36) (end 84.455 84.550991) (width 0.25) (layer "F.Cu") (net 39))
-  (segment (start 59.203299 50.12) (end 57.785 51.538299) (width 0.25) (layer "F.Cu") (net 39))
-  (segment (start 60.865 50.12) (end 59.203299 50.12) (width 0.25) (layer "F.Cu") (net 39))
   (segment (start 68.05 84.125) (end 65.815 86.36) (width 0.25) (layer "In1.Cu") (net 40))
   (segment (start 59.1 47.58) (end 60.865 47.58) (width 0.25) (layer "In1.Cu") (net 40))

Commit message: Update
Parts:
- moved C1 3.17 mm to (114.3, 79.4)
- moved C3 2.22 mm to (110.5, 79.4)
- moved C2 1.27 mm to (106.7, 79.4)
Routing:
- net VCC: track 231.2 -> 235.0 mm
- net GND: track 221.7 -> 219.1 mm
- net Reset: track 106.2 -> 104.3 mm
Other:
- board size 67.3 x 59.1 mm -> 62.9 x 59.1 mm
Changed lines of the file:
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@@
   )
   (footprint "Capacitor_THT:C_Rect_L4.0mm_W2.5mm_P2.50mm" (layer "F.Cu")
-    (at 112.7125 79.355 90)
+    (at 110.49 79.355 90)
     (descr "C, Rect series, Radial, pin pitch=2.50mm, , length*width=4*2.5mm^2, Capacitor")
     (tags "C Rect series Radial pin pitch 2.50mm  length 4mm width 2.5mm Capacitor")
@@
   )
   (footprint "Capacitor_THT:C_Rect_L4.0mm_W2.5mm_P2.50mm" (layer "F.Cu")
-    (at 117.475 79.355 90)
+    (at 114.3 79.355 90)
     (descr "C, Rect series, Radial, pin pitch=2.50mm, , length*width=4*2.5mm^2, Capacitor")
     (tags "C Rect series Radial pin pitch 2.50mm  length 4mm width 2.5mm Capacitor")
@@
   )
   (footprint "Capacitor_THT:C_Rect_L4.0mm_W2.5mm_P2.50mm" (layer "F.Cu")
-    (at 107.95 79.335 90)
+    (at 106.68 79.355 90)
     (descr "C, Rect series, Radial, pin pitch=2.50mm, , length*width=4*2.5mm^2, Capacitor")
     (tags "C Rect series Radial pin pitch 2.50mm  length 4mm width 2.5mm Capacitor")
@@
     )
   )
-  (gr_line (start 57.15 91.44) (end 120.65 91.44) (layer "Edge.Cuts") (width 0.1))
   (gr_line (start 54.61 33.655) (end 54.61 90.17) (layer "Edge.Cuts") (width 0.1))
+  (gr_line (start 57.15 91.44) (end 116.205 91.44) (layer "Edge.Cuts") (width 0.1))
   (gr_circle (center 57.15 88.9) (end 57.15 90.17) (layer "Edge.Cuts") (width 0.1) (fill none))
-  (gr_circle (center 119.38 88.9) (end 119.38 90.17) (layer "Edge.Cuts") (width 0.1) (fill none))
   (gr_line (start 55.88 91.44) (end 57.15 91.44) (layer "Edge.Cuts") (width 0.1))
-  (gr_arc (start 121.92 90.17) (mid 121.548026 91.068026) (end 120.65 91.44) (layer "Edge.Cuts") (width 0.1))
+  (gr_arc locked (start 117.475 90.17) (mid 117.103026 91.068026) (end 116.205 91.44) (layer "Edge.Cuts") (width 0.1))
   (gr_arc (start 54.61 33.655) (mid 54.981974 32.756974) (end 55.88 32.385) (layer "Edge.Cuts") (width 0.1))
-  (gr_arc (start 120.65 32.385) (mid 121.548026 32.756974) (end 121.92 33.655) (layer "Edge.Cuts") (width 0.1))
-  (gr_circle (center 119.38 34.925) (end 119.38 36.195) (layer "Edge.Cuts") (width 0.1) (fill none))
-  (gr_line (start 121.92 90.17) (end 121.92 33.655) (layer "Edge.Cuts") (width 0.1))
+  (gr_arc locked (start 116.205 32.385) (mid 117.103026 32.756974) (end 117.475 33.655) (layer "Edge.Cuts") (width 0.1))
+  (gr_line locked (start 117.475 90.17) (end 117.475 33.655) (layer "Edge.Cuts") (width 0.1))
   (gr_line (start 55.88 32.385) (end 57.15 32.385) (layer "Edge.Cuts") (width 0.1))
-  (gr_line (start 57.15 32.385) (end 120.65 32.385) (layer "Edge.Cuts") (width 0.1))
+  (gr_line (start 57.15 32.385) (end 116.205 32.385) (layer "Edge.Cuts") (width 0.1))
   (gr_arc (start 55.88 91.44) (mid 54.981974 91.068026) (end 54.61 90.17) (layer "Edge.Cuts") (width 0.1))
   (gr_text "CPU and paged RAM module" (at 95.25 60.96 90) (layer "B.SilkS")
@@
     (effects (font (size 1 1) (thickness 0.15)))
   )
+  (segment (start 111.115 70.495) (end 114.9775 70.495) (width 0.25) (layer "F.Cu") (net 1))
+  (segment (start 106.68 79.355) (end 105.41 78.085) (width 0.25) (layer "F.Cu") (net 1))
+  (segment (start 105.41 78.085) (end 105.41 76.2) (width 0.25) (layer "F.Cu") (net 1))
   (segment (start 106.68 53.95) (end 106.68 46.355) (width 0.25) (layer "F.Cu") (net 1))
-  (segment (start 114.9775 76.8575) (end 114.9775 70.495) (width 0.25) (layer "F.Cu") (net 1))
-  (segment (start 117.475 79.355) (end 114.9775 76.8575) (width 0.25) (layer "F.Cu") (net 1))
+  (segment (start 106.68 79.355) (end 114.3 79.355) (width 0.25) (layer "F.Cu") (net 1))
+  (segment (start 105.41 76.2) (end 111.115 70.495) (width 0.25) (layer "F.Cu") (net 1))
   (segment (start 106.68 54.5775) (end 106.68 53.95) (width 0.25) (layer "In1.Cu") (net 1))
   (segment (start 114.9775 62.875) (end 106.68 54.5775) (width 0.25) (layer "In1.Cu") (net 1))
@@
   (segment (start 60.428299 33.655) (end 100.48 33.655) (width 0.25) (layer "In2.Cu") (net 1))
   (segment (start 63.165 85.25) (end 74.545 85.25) (width 0.25) (layer "In2.Cu") (net 1))
-  (segment (start 117.455 79.335) (end 117.475 79.355) (width 0.25) (layer "In2.Cu") (net 1))
   (segment (start 62.23 84.315) (end 60.865 82.95) (width 0.25) (layer "In2.Cu") (net 1))
   (segment (start 60.865 82.95) (end 58.82 82.95) (width 0.25) (layer "In2.Cu") (net 1))
   (segment (start 100.48 33.655) (end 102.69 35.865) (width 0.25) (layer "In2.Cu") (net 1))
   (segment (start 58.82 82.95) (end 57.15 81.28) (width 0.25) (layer "In2.Cu") (net 1))
-  (segment (start 107.95 79.335) (end 117.455 79.335) (width 0.25) (layer "In2.Cu") (net 1))
   (segment (start 114.9775 62.875) (end 114.9775 70.495) (width 0.25) (layer "In2.Cu") (net 1))
   (segment (start 57.15 36.933299) (end 60.428299 33.655) (width 0.25) (layer "In2.Cu") (net 1))
@@
   (segment (start 106.35 40.945) (end 106.68 41.275) (width 0.25) (layer "F.Cu") (net 2))
   (segment (start 102.69 40.945) (end 106.35 40.945) (width 0.25) (layer "F.Cu") (net 2))
+  (segment (start 106.68 76.855) (end 114.3 76.855) (width 0.25) (layer "F.Cu") (net 2))
   (segment (start 83.29 63.805) (end 86.325 66.84) (width 0.25) (layer "F.Cu") (net 2))
   (segment (start 84.415 62.68) (end 87.815 62.68) (width 0.25) (layer "In1.Cu") (net 2))
@@
   (segment (start 83.29 63.805) (end 84.415 62.68) (width 0.25) (layer "In1.Cu") (net 2))
   (segment (start 101.565 48.099009) (end 102.514009 47.15) (width 0.25) (layer "In1.Cu") (net 2))
-  (segment (start 107.95 76.835) (end 117.455 76.835) (width 0.25) (layer "In2.Cu") (net 2))
-  (segment (start 117.475 76.855) (end 118.6 77.98) (width 0.25) (layer "In2.Cu") (net 2))
+  (segment (start 116.185 78.74) (end 114.3 76.855) (width 0.25) (layer "In2.Cu") (net 2))
   (segment (start 95.555 73.965) (end 107.875 86.285) (width 0.25) (layer "In2.Cu") (net 2))
+  (segment (start 116.205 86.78) (end 116.205 78.74) (width 0.25) (layer "In2.Cu") (net 2))
   (segment (start 59.69 84.315) (end 63.985 88.61) (width 0.25) (layer "In2.Cu") (net 2))
-  (segment (start 118.6 84.385) (end 114.375 88.61) (width 0.25) (layer "In2.Cu") (net 2))
+  (segment (start 116.205 78.74) (end 116.185 78.74) (width 0.25) (layer "In2.Cu") (net 2))
   (segment (start 107.875 86.285) (end 107.875 88.61) (width 0.25) (layer "In2.Cu") (net 2))
-  (segment (start 118.6 77.98) (end 118.6 84.385) (width 0.25) (layer "In2.Cu") (net 2))
-  (segment (start 117.455 76.835) (end 117.475 76.855) (width 0.25) (layer "In2.Cu") (net 2))
+  (segment (start 114.375 88.61) (end 116.205 86.78) (width 0.25) (layer "In2.Cu") (net 2))
   (segment (start 107.875 88.61) (end 114.375 88.61) (width 0.25) (layer "In2.Cu") (net 2))
   (segment (start 87.45 73.965) (end 95.555 73.965) (width 0.25) (layer "In2.Cu") (net 2))
@@
   (segment (start 63.955 52.66) (end 68.05 48.565) (width 0.25) (layer "F.Cu") (net 3))
   (segment (start 57.785 53.79) (end 58.915 52.66) (width 0.25) (layer "F.Cu") (net 3))
-  (segment (start 118.6 79.885) (end 118.6 50.655) (width 0.25) (layer "F.Cu") (net 4))
-  (segment (start 114.375 84.11) (end 118.6 79.885) (width 0.25) (layer "F.Cu") (net 4))
-  (segment (start 118.6 50.655) (end 114.3 46.355) (width 0.25) (layer "F.Cu") (net 4))
+  (segment (start 114.375 84.11) (end 116.205 82.28) (width 0.25) (layer "F.Cu") (net 4))
+  (segment (start 116.205 48.26) (end 114.3 46.355) (width 0.25) (layer "F.Cu") (net 4))
+  (segment (start 116.205 82.28) (end 116.205 48.26) (width 0.25) (layer "F.Cu") (net 4))
   (segment (start 83.29 71.425) (end 85.859009 71.425) (width 0.25) (layer "In2.Cu") (net 4))
   (segment (start 93.775 70.01) (end 107.556802 83.791802) (width 0.25) (layer "In2.Cu") (net 4))

Commit message: Final before order
Parts:
- removed R13: 10K, Resistor_THT:R_Axial_DIN0204_L3.6mm_D1.6mm_P7.62mm_Horizontal
- added U1: 74LS32, Package_DIP:DIP-14_W7.62mm_Socket, F.Cu at (107.3, 36.2)
- SW2: value SW_DIP_x04 -> SW_DIP_x03; footprint Button_Switch_THT:SW_DIP_SPSTx04_Slide_9.78x12.34mm_W7.62mm_P2.54mm -> Button_Switch_THT:SW_DIP_SPSTx03_Slide_9.78x9.8mm_W7.62mm_P2.54mm
- moved R12 52.2 mm to (90.2, 85.7), turned to 90 degrees
- moved R14 50.7 mm to (87.6, 85.7), turned to 90 degrees
- moved R15 44.2 mm to (92.7, 85.7), turned to 90 degrees
- moved R9 41.0 mm to (95.2, 85.7), turned to 90 degrees
- moved R2 37.9 mm to (97.8, 85.7), turned to 90 degrees
- moved R1 34.9 mm to (100.3, 85.7), turned to 90 degrees
- moved R3 32.0 mm to (102.8, 85.7), turned to 90 degrees
- moved SW1 14.6 mm to (107.2, 75.9), turned to 0 degrees
- moved C1 8.87 mm to (114.3, 70.5)
- moved C2 8.87 mm to (106.7, 70.5)
- moved C3 8.87 mm to (110.5, 70.5)
- moved SW2 5.11 mm to (106.7, 57.8)
Connections:
- R12 pad 2: /A12 -> /A15
- R14 pad 2: /A11 -> /A14
- R15 pad 2: /A13 -> /A16
- SW2 pad 1: /A11 -> /A14
- SW2 pad 2: /A12 -> /A15
- SW2 pad 3: /A13 -> /A16
- SW2 pad 4: /A14 -> VCC
- U3 pad 1: GND -> unconnected-(U3-Pad1)
- U3 pad 2: GND -> /A16
- U3 pad 22: MREQ -> Net-(U3-Pad22)
- U3 pad 24: RD -> OE
- U3 pad 3: GND -> /A15
- U3 pad 30: GND -> unconnected-(U3-Pad30)
Routing:
- net /A15: track 10.4 -> 108.6 mm
- net GND: track 219.1 -> 134.6 mm
- net /A12: track 113.5 -> 40.9 mm
- net /A16: track 0.00 -> 69.3 mm
- net BRQ: track 130.1 -> 68.8 mm
- net Reset: track 104.3 -> 62.0 mm
- net /A13: track 92.7 -> 50.7 mm
- net INT: track 116.5 -> 75.3 mm
- net NMI: track 110.7 -> 77.5 mm
- net /A11: track 99.1 -> 67.3 mm
- net Net-(U3-Pad22): track 0.00 -> 23.0 mm
- net MREQ: track 106.3 -> 87.0 mm
- net /A14: track 86.2 -> 105.1 mm
- net /D3: track 84.3 -> 68.8 mm
- net /D6: track 67.0 -> 52.7 mm
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Other:
- board size 62.9 x 59.1 mm -> 62.9 x 55.6 mm
