File: modules/CpuRamModule/CpuRamModule.kicad_sch (KiCad schematic)
At the start: 16 parts, among them J1 Conn_02x20_Odd_Even, SW1 SW_Push, SW2 SW_DIP_x04, U2 Z80CPU, U3 SST39SF010

Commit message: Final before order
Parts:
- removed R13: 10K, Resistor_THT:R_Axial_DIN0204_L3.6mm_D1.6mm_P7.62mm_Horizontal, symbol Device:R
- removed SW2: SW_DIP_x04, Button_Switch_THT:SW_DIP_SPSTx04_Slide_9.78x12.34mm_W7.62mm_P2.54mm, symbol Switch:SW_DIP_x04
- added SW2: SW_DIP_x03, Button_Switch_THT:SW_DIP_SPSTx03_Slide_9.78x9.8mm_W7.62mm_P2.54mm, symbol Switch:SW_DIP_x03
- added U1: 74LS32, Package_DIP:DIP-14_W7.62mm_Socket, symbol 74xx:74LS32
Connections:
- net A11: no longer R14.2
- net A12: no longer R12.2
- net A13: no longer R15.2
- net A14: now also R14.2, SW2.1, U1.1
- net A15: now also R12.2, U3.3 (A15), SW2.2, U1.2
- net GND: now also U1.7 (GND); no longer U3.1 (NC), U3.2 (A16), U3.3 (A15), U3.30 (NC)
- net MREQ: now also U1.5; no longer U3.22 (CE)
- net RD: now also U1.4; no longer U3.24 (OE)
- net VCC: now also SW2.4, SW2.5, SW2.6, U1.14 (VCC)
- new net: U1.3, U3.22 (CE)
- new net A16: R15.2, SW2.3, U3.2 (A16)
- new net OE: U1.6, U3.24 (OE)
Other:
- moved on the sheet: R12, R14, R15, R9, SW1
